File: kicad/electronics/electronics.kicad_sch (KiCad schematic)
At the start: 15 parts

Commit message: Added power switch to schematic
Parts:
- added SW?: SW_SPST, symbol Switch:SW_SPST
Connections:
- net GND: now also SW?.1 (A)
- net enable: now reaches A?.27 (EN)
- net enable: now also SW?.2 (B)
Other:
- note added: "Power Switch"
Changed lines of the file:
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@@
+    (stroke (width 0) (type default) (color 0 0 0 0))
+  )
+  (wire (pts (xy 186.69 104.14) (xy 190.5 104.14))
     (stroke (width 0) (type default) (color 0 0 0 0))
   )
@@
     (stroke (width 0) (type default) (color 0 0 0 0))
   )
+  (wire (pts (xy 173.99 104.14) (xy 176.53 104.14))
+    (stroke (width 0) (type default) (color 0 0 0 0))
+  )
   (wire (pts (xy 24.13 54.61) (xy 24.13 66.04))
     (stroke (width 0) (type default) (color 0 0 0 0))
@@
     (stroke (width 0) (type default) (color 0 0 0 0))
   )
+  (polyline (pts (xy 171.45 90.17) (xy 171.45 111.76))
+    (stroke (width 0) (type default) (color 0 0 0 0))
+  )
   (wire (pts (xy 38.1 77.47) (xy 38.1 78.74))
     (stroke (width 0) (type default) (color 0 0 0 0))
@@
     (stroke (width 0) (type default) (color 0 0 0 0))
   )
+  (polyline (pts (xy 200.66 111.76) (xy 171.45 111.76))
+    (stroke (width 0) (type default) (color 0 0 0 0))
+  )
   (wire (pts (xy 77.47 43.18) (xy 90.17 43.18))
     (stroke (width 0) (type default) (color 0 0 0 0))
@@
     (stroke (width 0) (type default) (color 0 0 0 0))
   )
+  (polyline (pts (xy 200.66 90.17) (xy 200.66 111.76))
+    (stroke (width 0) (type default) (color 0 0 0 0))
+  )
   (wire (pts (xy 160.02 49.53) (xy 163.83 49.53))
     (stroke (width 0) (type default) (color 0 0 0 0))
@@
   )
   (wire (pts (xy 115.57 66.04) (xy 124.46 66.04))
+    (stroke (width 0) (type default) (color 0 0 0 0))
+  )
+  (polyline (pts (xy 171.45 90.17) (xy 200.66 90.17))
+    (stroke (width 0) (type default) (color 0 0 0 0))
+  )
+  (wire (pts (xy 115.57 45.72) (xy 124.46 45.72))
     (stroke (width 0) (type default) (color 0 0 0 0))
   )
@@
     (effects (font (size 1.27 1.27)) (justify left bottom))
   )
+  (text "Power Switch" (at 172.72 93.98 0)
+    (effects (font (size 1.27 1.27)) (justify left bottom))
+  )
   (text "buzzer" (at 147.32 93.98 0)
     (effects (font (size 1.27 1.27)) (justify left bottom))
@@
     )
   )
+  (global_label "enable" (shape input) (at 124.46 45.72 0) (fields_autoplaced)
+    (effects (font (size 1.27 1.27)) (justify left))
+    (property "Intersheet References" "${INTERSHEET_REFS}" (id 0) (at 133.1626 45.6406 0)
+      (effects (font (size 1.27 1.27)) (justify left) hide)
+    )
+  )
   (global_label "usd_miso" (shape input) (at 237.49 39.37 0) (fields_autoplaced)
     (effects (font (size 1.27 1.27)) (justify left))
@@
     (property "Intersheet References" "${INTERSHEET_REFS}" (id 0) (at 66.2879 63.4206 0)
       (effects (font (size 1.27 1.27)) (justify right) hide)
+    )
+  )
+  (global_label "enable" (shape input) (at 190.5 104.14 0) (fields_autoplaced)
+    (effects (font (size 1.27 1.27)) (justify left))
+    (property "Intersheet References" "${INTERSHEET_REFS}" (id 0) (at 199.2026 104.0606 0)
+      (effects (font (size 1.27 1.27)) (justify left) hide)
     )
   )
@@
     (pin "1")
   )
+  (symbol (lib_id "power:GND") (at 173.99 104.14 0) (unit 1)
+    (in_bom yes) (on_board yes) (fields_autoplaced)
+    (property "Reference" "#PWR?" (id 0) (at 173.99 110.49 0)
+      (effects (font (size 1.27 1.27)) hide)
+    )
+    (property "Value" "GND" (id 1) (at 173.99 109.22 0))
+    (property "Footprint" "" (id 2) (at 173.99 104.14 0)
+      (effects (font (size 1.27 1.27)) hide)
+    )
+    (property "Datasheet" "" (id 3) (at 173.99 104.14 0)
+      (effects (font (size 1.27 1.27)) hide)
+    )
+    (pin "1")
+  )
   (symbol (lib_id "power:+3V3") (at 189.23 62.23 0) (unit 1)
     (in_bom yes) (on_board yes) (fields_autoplaced)
@@
     )
     (pin "1")
+  )
+  (symbol (lib_id "Switch:SW_SPST") (at 181.61 104.14 0) (unit 1)
+    (in_bom yes) (on_board yes) (fields_autoplaced)
+    (property "Reference" "SW?" (id 0) (at 181.61 97.79 0))
+    (property "Value" "SW_SPST" (id 1) (at 181.61 100.33 0))
+    (property "Footprint" "" (id 2) (at 181.61 104.14 0)
+      (effects (font (size 1.27 1.27)) hide)
+    )
+    (property "Datasheet" "~" (id 3) (at 181.61 104.14 0)
+      (effects (font (size 1.27 1.27)) hide)
+    )
+    (pin "1")
+    (pin "2")
   )
   (symbol (lib_id "MCU_Module:Adafruit_Feather_HUZZAH32_ESP32") (at 102.87 58.42 0) (unit 1)
@@
       (reference "#PWR?") (unit 1) (value "+3V3") (footprint "")
     )
+    (path "/474d4243-235c-488b-86c1-9613c3d59f32"
+      (reference "#PWR?") (unit 1) (value "GND") (footprint "")
+    )
     (path "/580001aa-8235-48fc-87c7-a847444586c6"
       (reference "#PWR?") (unit 1) (value "+3V3") (footprint "")
@@
       (reference "R?") (unit 1) (value "1k") (footprint "")
     )
+    (path "/b4e38075-0bc2-4a06-8645-00981208636e"
+      (reference "SW?") (unit 1) (value "SW_SPST") (footprint "")
+    )
     (path "/d4f7f3b1-0ecb-4ccb-b494-536334ef8eaa"
